Commit message: second_day

File: my_model/urdf/robo_robot.urdf (robot description, URDF)
Before this commit: robot r2d2, 11 links, 10 joints
Links:
- link caster_front_link: mass 0.05 -> 0.5
- link caster_link: geometry collision cylinder length=0.02586 radius=0.005; visual cylinder length=0.02586 radius=0.01214
Joints:
- joint caster_front_joint: axis 0 0 0 -> 0 1 0; type continuous -> fixed
- joint caster_front_joint_base: origin xyz=0 0.0 -0.01545 rpy=0 0 0 -> xyz=0 0.0 -0.00545 rpy=0 0 0
- joint laser_sensor: origin xyz=0.05 0 0.015 rpy=0 0.05 0 -> xyz=0.05 0 0.015 rpy=0 0 0
- joint left_wheel_joint: origin xyz=-0.09 -0.095 0 rpy=0 0 0 -> xyz=-0.06 -0.095 0 rpy=0 0 0
- joint right_wheel_joint: origin xyz=-0.09 0.095 0 rpy=0 0 0 -> xyz=-0.06 0.095 0 rpy=0 0 0

Commit message: final_submission

File: my_model/urdf/robo_robot.urdf (robot description, URDF)
Before this commit: robot r2d2, 11 links, 10 joints
Links:
- removed link base_upperlink
- removed link support_1
- removed link support_2
- removed link support_3
- removed link support_4
- link base_link: geometry collision cylinder length=0.005 radius=0.08; visual cylinder length=0.004 radius=0.08
- link left_wheel: mass 0.05 -> 0.5; geometry collision cylinder length=0.005 radius=0.025; visual cylinder length=0.02 radius=0.0325
- link right_wheel: mass 0.05 -> 0.5; geometry collision cylinder length=0.005 radius=0.025; visual cylinder length=0.02 radius=0.0325
Joints:
- removed joint base_upperlink_joint
- removed joint support_joint1
- removed joint support_joint2
- removed joint support_joint3
- removed joint support_joint4
- joint caster_front_joint: type fixed -> continuous
- joint laser_sensor: origin xyz=0.05 0 0.015 rpy=0 0 0 -> xyz=0.05 0 0.015 rpy=0 .02 0
- joint left_wheel_joint: origin xyz=-0.06 -0.095 0 rpy=0 0 0 -> xyz=-0.03 -0.09 0 rpy=0 0 0
- joint right_wheel_joint: origin xyz=-0.06 0.095 0 rpy=0 0 0 -> xyz=-0.03 0.09 0 rpy=0 0 0
